Commit message: update inertia and mass

File: aero_shop/hand_yaw/urdf/hand_yaw.urdf.xacro (robot description, xacro)
@@ -25,11 +25,7 @@
     </collision> </xacro:unless>
     <inertial>
-      <mass value="0.183" />
-      <!-- original version -->
-      <!--origin xyz="0 0 -0.0875" rpy="0 -0 0"/>
-      <inertia ixx="0.000601" ixy="0" ixz="0" iyy="0.00055" iyz="0" izz="0.000102"/-->
-      <!-- just fixed for gazebo / aim to increase z axis inertia-->
-      <origin xyz="0 0.014 -0.02" rpy="0 -0 0"/>
-      <inertia ixx="0.0005" ixy="0" ixz="0" iyy="0.0005" iyz="0" izz="0.0007" />
+      <mass value="0.3115" />
+      <origin xyz="0.0097 ${reflect * 0.0003} -0.0413" rpy="0 -0 0"/>
+      <inertia ixx="0.0001" ixy="0" ixz="0.0001" iyy="0.0002" iyz="0" izz="0.0002" />
     </inertial>
   </link>

File: aero_shop/typeC_lifter/urdf/lifter.urdf.xacro (robot description, xacro)
@@ -32,7 +32,7 @@
       </collision>
       <inertial>
-        <mass value="7.64604" />
-        <origin xyz="-0.012819 -0.002679 0.007207" rpy="0 -0 0"/>
-        <inertia ixx="0.0658136" ixy="-0.000159462" ixz="0.010103" iyy="0.0504268" iyz="0.000173435" izz="0.0889772"/>
+        <mass value="1.074" />
+        <origin xyz="0.004 0.0 0.044" rpy="0 0 0"/>
+        <inertia ixx="0.004" ixy="0.0" ixz="0.0" iyy="0.001" iyz="0.0" izz="0.002"/>
       </inertial>
     </link>
@@ -52,9 +52,7 @@
       </collision>
       <inertial>
-        <mass value="2.06679" />
-        <!--origin xyz="0.081713 0.000812 -0.146934" rpy="0 -0 0"/-->
-        <origin xyz="0.051713 0.0 0.146934" rpy="0 -0 0"/>
-        <!--inertia ixx="0.0408818" ixy="-9.39301e-06" ixz="-0.000750165" iyy="0.0403969" iyz="-0.000120419" izz="0.00260982"/-->
-        <inertia ixx="0.06" ixy="0.0" ixz="0.0" iyy="0.1" iyz="0.0" izz="0.06"/>
+        <mass value="1.221" />
+        <origin xyz="0.003 0 0.107" rpy="0 0 0"/>
+        <inertia ixx="0.006" ixy="0.0" ixz="0.0" iyy="0.006" iyz="0.0" izz="0.002"/>
       </inertial>
     </link>
@@ -74,9 +72,7 @@
       </collision>
       <inertial>
-        <mass value="2.06679" />
-        <!--origin xyz="0.081713 0.000812 -0.146934" rpy="0 -0 0"/-->
-        <origin xyz="-0.031713 0.0 0.046934" rpy="0 -0 0"/>
-        <!--inertia ixx="0.0408818" ixy="-9.39301e-06" ixz="-0.000750165" iyy="0.0403969" iyz="-0.000120419" izz="0.00260982"/-->
-        <inertia ixx="0.06" ixy="0.0" ixz="0.0" iyy="0.1" iyz="0.0" izz="0.06"/>
+        <mass value="0.829" />
+        <origin xyz="-0.004 0.0 0.06" rpy="0 0 0"/>
+        <inertia ixx="0.003" ixy="0.0" ixz="0.0" iyy="0.003" iyz="0.0" izz="0.001"/>
       </inertial>
     </link>
@@ -96,8 +92,8 @@
       </collision>
       <inertial>
-        <mass value="2.62321" />
-        <!--origin xyz="0.0587169 0 -0.135292" rpy="0 -0 0"/-->
-        <origin xyz="-0.0587169 0 0.135292" rpy="0 -0 0"/>
-        <inertia ixx="0.0161595" ixy="-9.27234e-05" ixz="0.00262839" iyy="0.0166415" iyz="-0.00017447" izz="0.00477281"/>
+        <mass value="1.221" />
+        <mass value="0" />
+        <origin xyz="0.003 0 0.143" rpy="0 0 0"/>
+        <inertia ixx="0.006" ixy="0.0" ixz="0.0" iyy="0.006" iyz="0.0" izz="0.002"/>
       </inertial>
     </link>
@@ -105,19 +101,19 @@
     <link name="leg_base_link">
       <visual>
-        <origin xyz="0 0 0.05" rpy="3.1415920 0 0"/>
-        <geometry>
-          <mesh filename="package://aero_description/meshes/typeC_lifter/lifter_base.dae" scale="1 1 1" />
-        </geometry>
-      </visual>
-      <collision>
-        <origin xyz="0 0 0.05" rpy="3.1415920 0 0"/>
-        <geometry>
-          <mesh filename="package://aero_description/meshes/typeC_lifter/lifter_base.dae" scale="1 1 1" />
-        </geometry>
-      </collision>
-      <inertial>
-        <mass value="7.64604" />
-        <origin xyz="-0.012819 -0.002679 0.007207" rpy="0 -0 0"/>
-        <inertia ixx="0.0658136" ixy="-0.000159462" ixz="0.010103" iyy="0.0504268" iyz="0.000173435" izz="0.0889772"/>
+        <origin xyz="0 0 0.05" rpy="3.1415 0 0"/>
+        <geometry>
+          <mesh filename="package://aero_description/meshes/typeC_lifter/lifter_base.dae" scale="1 1 1" />
+        </geometry>
+      </visual>
+      <collision>
+        <origin xyz="0 0 0.05" rpy="3.1415 0 0"/>
+        <geometry>
+          <mesh filename="package://aero_description/meshes/typeC_lifter/lifter_base.dae" scale="1 1 1" />
+        </geometry>
+      </collision>
+      <inertial>
+        <mass value="1.074" />
+        <origin xyz="0.004 0.0 -0.044" rpy="0 0 0"/>
+        <inertia ixx="0.002" ixy="0.0" ixz="0.0" iyy="0.001" iyz="0.0" izz="0.002"/>
       </inertial>
     </link>
@@ -137,7 +133,7 @@
       </collision>
       <inertial>
-        <mass value="1.0" />
-        <origin xyz="0.0 0.0 0.0" rpy="0 0 0"/>
-        <inertia ixx="0.03" ixy="0.0" ixz="0.0" iyy="0.03" iyz="0.0" izz="0.04"/>
+        <mass value="0.82" />
+        <origin xyz="-0.002 0.0 0.0" rpy="0 0 0"/>
+        <inertia ixx="0.003" ixy="0.0" ixz="0.0" iyy="0.002" iyz="0.0" izz="0.005"/>
       </inertial>
     </link>
@@ -192,7 +188,7 @@
       </visual>
       <inertial> <!-- for gazebo visualization -->
-        <mass value="0.4"/>
-        <origin rpy="0 0 0" xyz="-0.04 0.0 0.14"/>
-        <inertia ixx="0.001" ixy="0" ixz="0" iyy="0.001" iyz="0" izz="0.001"/>
+        <mass value="0.376"/>
+        <origin rpy="0 0 0" xyz="0.011 0.0 0.129"/>
+        <inertia ixx="0.0025" ixy="0.0" ixz="0.0021" iyy="0.008" iyz="0" izz="0.0005"/>
       </inertial>
     </link>
@@ -205,7 +201,7 @@
       </visual>
       <inertial> <!-- for gazebo visualization -->
-        <mass value="0.4"/>
-        <origin rpy="0 0 0" xyz="-0.04 0.0 0.14"/>
-        <inertia ixx="0.001" ixy="0" ixz="0" iyy="0.001" iyz="0" izz="0.001"/>
+        <mass value="0.376"/>
+        <origin rpy="0 0 0" xyz="0.011 0.0 0.129"/>
+        <inertia ixx="0.0025" ixy="0.0" ixz="0.0021" iyy="0.008" iyz="0" izz="0.0005"/>
       </inertial>
     </link>

File: aero_shop/typeE_wheel/urdf/wheels.urdf.xacro (robot description, xacro)
@@ -38,7 +38,7 @@
       </collision> </xacro:unless>
       <inertial>
-        <mass value="70" />
-        <origin xyz="0 0 0.04" rpy="0 -0 0.0"/>
-        <inertia ixx="0.528" ixy="0" ixz="0" iyy="2.02" iyz="0" izz="2.35"/>
+        <mass value="19.633" />
+        <origin xyz="-0.035 0 0.016" rpy="0 0 0.0"/>
+        <inertia ixx="0.325" ixy="0.002" ixz="0.016" iyy="1.018" iyz="0" izz="1.260"/>
       </inertial>
     </link>
@@ -53,7 +53,7 @@
       <!-- no collision geometry -->
       <inertial>
-        <mass value="1" />
+        <mass value="2.755" />
         <origin xyz="0 0 0" rpy="0 -0 0"/>
-        <inertia ixx="0.528" ixy="0" ixz="0" iyy="2.02" iyz="0" izz="2.35"/>
+        <inertia ixx="0.025" ixy="0" ixz="0" iyy="0.004" iyz="0" izz="0.027"/>
       </inertial>
     </link>
@@ -74,7 +74,7 @@
       </collision> </xacro:unless>
       <inertial>
-        <mass value="1" />
-        <origin xyz="0 0 0" rpy="0 -0 0"/>
-        <inertia ixx="0.528" ixy="0" ixz="0" iyy="2.02" iyz="0" izz="2.35"/>
+        <mass value="0.6" />
+        <origin xyz="0 0 0" rpy="0 0 0"/>
+        <inertia ixx="0.001" ixy="0" ixz="0" iyy="0.001" iyz="0" izz="0.002"/>
       </inertial>
     </link>
@@ -95,7 +95,7 @@
       </collision> </xacro:unless>
       <inertial>
-        <mass value="1" />
-        <origin xyz="0 0 0" rpy="0 -0 0"/>
-        <inertia ixx="0.528" ixy="0" ixz="0" iyy="2.02" iyz="0" izz="2.35"/>
+        <mass value="0.6" />
+        <origin xyz="0 0 0" rpy="0 0 0"/>
+        <inertia ixx="0.001" ixy="0" ixz="0" iyy="0.001" iyz="0" izz="0.002"/>
       </inertial>
     </link>
@@ -116,7 +116,7 @@
       </collision> </xacro:unless>
       <inertial>
-        <mass value="1" />
-        <origin xyz="0 0 0" rpy="0 -0 0"/>
-        <inertia ixx="0.528" ixy="0" ixz="0" iyy="2.02" iyz="0" izz="2.35"/>
+        <mass value="0.6" />
+        <origin xyz="0 0 0" rpy="0 0 0"/>
+        <inertia ixx="0.001" ixy="0" ixz="0" iyy="0.001" iyz="0" izz="0.002"/>
       </inertial>
     </link>
@@ -137,7 +137,7 @@
       </collision> </xacro:unless>
       <inertial>
-        <mass value="1" />
-        <origin xyz="0 0 0" rpy="0 -0 0"/>
-        <inertia ixx="0.528" ixy="0" ixz="0" iyy="2.02" iyz="0" izz="2.35"/>
+        <mass value="0.6" />
+        <origin xyz="0 0 0" rpy="0 0 0"/>
+        <inertia ixx="0.001" ixy="0" ixz="0" iyy="0.001" iyz="0" izz="0.002"/>
       </inertial>
     </link>
@@ -157,7 +157,7 @@
       </collision> </xacro:unless>
       <inertial>
-        <mass value="0.2" />
-        <origin xyz="0 0 0" rpy="0 -0 0"/>
-        <inertia ixx="0.0528" ixy="0" ixz="0" iyy="0.0202" iyz="0" izz="0.0235"/>
+        <mass value="0.1" />
+        <origin xyz="0 0 0" rpy="0 0 0"/>
+        <inertia ixx="0" ixy="0" ixz="0" iyy="0" iyz="0" izz="0"/>
       </inertial>
     </link>

File: aero_shop/typeF_upperbody/urdf/aero_upper_typef.urdf.xacro (robot description, xacro)
@@ -11,20 +11,13 @@
   <!-- ============================   aero(typeF_upper)   ============================ -->
   <link name="${base_link}">
-    <xacro:unless value="${disable_mesh}"> <visual>
-      <origin xyz="0 0 0" rpy="0 -0 0"/>
-      <geometry>
-        <mesh filename="package://aero_description/meshes/typeF_upperbody/WAIST_LINK0_mesh.dae" scale="1 1 1" />
-      </geometry>
-    </visual> </xacro:unless>
-    <xacro:unless value="${disable_mesh}"> <collision>
-      <origin xyz="0 0 0" rpy="0 -0 0"/>
-      <geometry>
-        <mesh filename="package://aero_description/meshes/typeF_upperbody/WAIST_LINK0_mesh.dae" scale="1 1 1" />
-      </geometry>
-    </collision> </xacro:unless>
-    <inertial>
-      <mass value="1.257" />
-      <origin xyz="0 0 0.0" rpy="0 -0 0"/>
-      <inertia ixx="0.034" ixy="0" ixz="0" iyy="0.034" iyz="0" izz="0.018"/>
+    <inertial>
+<!--
+        <mass value="0.82" />
+        <origin xyz="-0.002 0.0 0.0" rpy="0 0 0"/>
+        <inertia ixx="0.003" ixy="0.0" ixz="0.0" iyy="0.002" iyz="0.0" izz="0.005"/>
+-->
+        <mass value="0.001" />
+        <origin xyz="0.0 0.0 0.0" rpy="0 0 0"/>
+        <inertia ixx="0.0" ixy="0.0" ixz="0.0" iyy="0.0" iyz="0.0" izz="0.0"/>
     </inertial>
   </link>
@@ -44,9 +37,7 @@
     </collision> </xacro:unless>
     <inertial>
-      <mass value="1.257" />
-      <origin xyz="0 0 0.042" rpy="0 -0 0"/>
-      <!-- inertia ixx="0.034" ixy="0" ixz="0" iyy="0.034" iyz="0" izz="0.018"/ -->
-      <!-- just fixed for gazebo / reduce inertia-->
-      <inertia ixx="0.01" ixy="0" ixz="0" iyy="0.01" iyz="0" izz="0.007"/>
+      <mass value="1.105" />
+      <origin xyz="0.001 0.0 0.064" rpy="0 -0 0"/>
+      <inertia ixx="0.0026" ixy="0" ixz="0" iyy="0.0026" iyz="0" izz="0.0013"/>
     </inertial>
   </link>
@@ -54,9 +45,7 @@
   <link name="hip_center">
     <inertial>
-      <mass value="0.1" />
-      <origin xyz="0 0 0" rpy="0 -0 0"/>
-      <!--inertia ixx="0.01" ixy="0" ixz="0" iyy="0.01" iyz="0" izz="0.01"/-->
-      <!-- just fixed for gazebo / reduce inertia-->
-      <inertia ixx="0.003" ixy="0" ixz="0" iyy="0.003" iyz="0" izz="0.003"/>
+      <mass value="0.012" />
+      <origin xyz="0.0 0.0 0.0" rpy="0 -0 0"/>
+      <inertia ixx="0.0" ixy="0" ixz="0" iyy="0.0" iyz="0" izz="0.0"/>
     </inertial>
   </link>
@@ -76,7 +65,10 @@
     </collision> </xacro:unless>
     <inertial>
-      <mass value="10.551" />
-      <origin xyz="0 0 0.22" rpy="0 -0 0"/>
-      <inertia ixx="0.13" ixy="0" ixz="0" iyy="0.12" iyz="0" izz="0.114"/>
+      <mass value="6.7" />
+      <origin xyz="0.001 0 0.197" rpy="0 -0 0"/>
+<!--
+      <inertia ixx="0.334" ixy="0" ixz="0.0035" iyy="0.308" iyz="0.0001" izz="0.0497"/>
+-->
+      <inertia ixx="0.07378" ixy="0" ixz="0.0044" iyy="0.048" iyz="0.0001" izz="0.0497"/>
     </inertial>
   </link>
@@ -96,10 +88,7 @@
     </collision> </xacro:unless>
     <inertial>
-      <mass value="0.242" />
-      <!--origin xyz="0 0.02 0" rpy="0 -0 0"/>
-      <inertia ixx="0.000228" ixy="0" ixz="0" iyy="0.000148" iyz="0" izz="0.000263"/-->
-      <!-- just fixed for gazebo / increase inertia-->
-      <origin xyz="0 0.02 0.015" rpy="0 -0 0"/>
-      <inertia ixx="0.00133" ixy="0" ixz="0" iyy="0.001" iyz="0" izz="0.00133"/>
+      <mass value="0.738" />
+      <origin xyz="-0.0001 -0.0499 0.0044" rpy="0 -0 0"/>
+      <inertia ixx="0.002" ixy="0" ixz="0" iyy="0.0003" iyz="0.0002" izz="0.0019"/>
     </inertial>
   </link>
@@ -119,8 +108,7 @@
     </collision> </xacro:unless>
     <inertial>
-      <mass value="0.744" />
-      <!--origin xyz="0 0.01 0" rpy="0 -0 0"/-->
-      <origin xyz="0 -0.01 -0.06" rpy="0 -0 0"/>
-      <inertia ixx="0.000841" ixy="0" ixz="0" iyy="0.000835" iyz="0" izz="0.000304"/>
+      <mass value="0.834" />
+      <origin xyz="-0.0007 -0.0093 -0.0768" rpy="0 -0 0"/>
+      <inertia ixx="0.0011" ixy="0" ixz="0.0" iyy="0.0011" iyz="0" izz="0.0004"/>
     </inertial>
   </link>
@@ -140,10 +128,7 @@
     </collision> </xacro:unless>
     <inertial>
-      <mass value="0.574" />
-      <!--origin xyz="0.005 0 -0.0654" rpy="0 -0 0"/>
-      <inertia ixx="0.00114" ixy="0" ixz="0" iyy="0.00117" iyz="0" izz="0.000269"/-->
-      <!-- fix for gazebo -->
-      <origin xyz="0.005 0 -0.0654" rpy="0 -0 0"/>
-      <inertia ixx="0.00214" ixy="0" ixz="0" iyy="0.00217" iyz="0" izz="0.003"/>
+      <mass value="0.852" />
+      <origin xyz="-0.0099 0 -0.0496" rpy="0 -0 0"/>
+      <inertia ixx="0.0015" ixy="0" ixz="0.0001" iyy="0.0016" iyz="0" izz="0.0005"/>
     </inertial>
   </link>
@@ -163,10 +148,7 @@
     </collision> </xacro:unless>
     <inertial>
-      <mass value="0.711" />
-      <!--origin xyz="0.0047 0 -0.0546" rpy="0 -0 0"/>
-      <inertia ixx="0.00178" ixy="0" ixz="0" iyy="0.00179" iyz="0" izz="0.000273"/-->
-      <!-- fix for gazebo -->
-      <origin xyz="-0.03 0 -0.0546" rpy="0 -0 0"/>
-      <inertia ixx="0.00178" ixy="0" ixz="0" iyy="0.00179" iyz="0" izz="0.0035"/>
+      <mass value="0.251" />
+      <origin xyz="-0.0422 -0.0002 -0.0061" rpy="0 -0 0"/>
+      <inertia ixx="0.0005" ixy="0" ixz="0.0001" iyy="0.0005" iyz="0" izz="0.0002"/>
     </inertial>
   </link>
@@ -186,8 +168,7 @@
     </collision> </xacro:unless>
     <inertial>
-      <mass value="0.132" />
-      <origin xyz="0.006 0 -0.0738" rpy="0 -0 0"/>
-      <!--inertia ixx="0.00276" ixy="0" ixz="0" iyy="0.00286" iyz="0" izz="0.004"/-->
-      <inertia ixx="0.0007" ixy="0" ixz="0" iyy="0.0007" iyz="0" izz="0.0004"/>
+      <mass value="0.91" />
+      <origin xyz="0.0 0.0018 -0.0754" rpy="0 -0 0"/>
+      <inertia ixx="0.0022" ixy="0" ixz="0" iyy="0.0023" iyz="0" izz="0.0004"/>
     </inertial>
   </link>
@@ -195,7 +176,7 @@
   <link name="l_wrist_center">
     <inertial>
-      <mass value="0.05" />
-      <origin xyz="0 0 0" rpy="0 -0 0"/>
-      <inertia ixx="0.0001" ixy="0" ixz="0" iyy="0.0001" iyz="0" izz="0.0001"/>
+      <mass value="0.005" />
+      <origin xyz="0 -0.0019 0" rpy="0 -0 0"/>
+      <inertia ixx="0.0" ixy="0" ixz="0" iyy="0.0" iyz="0" izz="0.0"/>
     </inertial>
   </link>
@@ -215,8 +196,7 @@
     </collision> </xacro:unless>
     <inertial>
-      <mass value="0.341" />
-      <origin xyz="0 0 0.0595" rpy="0 -0 0"/>
-      <!--inertia ixx="1.64186e-35" ixy="0" ixz="0" iyy="1.64186e-35" iyz="0" izz="0"/-->
-      <inertia ixx="0.001" ixy="0" ixz="0" iyy="0.001" iyz="0" izz="0.002"/>
+      <mass value="0.275" />
+      <origin xyz="-0.0003 0.0003 0.0439" rpy="0 -0 0"/>
+      <inertia ixx="0.0002" ixy="0" ixz="0" iyy="0.0002" iyz="0" izz="0.0001"/>
     </inertial>
   </link>
@@ -236,7 +216,7 @@
     </collision> </xacro:unless>
     <inertial>
-      <mass value="0.1" />
-      <origin xyz="0 0 0" rpy="0 -0 0"/>
-      <inertia ixx="0.0005" ixy="0" ixz="0" iyy="0.0005" iyz="0" izz="0.0005"/>
+      <mass value="0.005" />
+      <origin xyz="0 -0.0019 0" rpy="0 -0 0"/>
+      <inertia ixx="0.00" ixy="0" ixz="0" iyy="0.0005" iyz="0" izz="0.0"/>
     </inertial>
   </link>
@@ -256,7 +236,7 @@
     </collision> </xacro:unless>
     <inertial>
-      <mass value="0.974" />
-      <origin xyz="0.01 0 0.070" rpy="0 -0 0"/>
-      <inertia ixx="0.005" ixy="0" ixz="0" iyy="0.005" iyz="0" izz="0.005"/>
+      <mass value="0.685" />
+      <origin xyz="0.0047 0 0.0711" rpy="0 -0 0"/>
+      <inertia ixx="0.0018" ixy="0" ixz="0.0001" iyy="0.0017" iyz="0" izz="0.0014"/>
     </inertial>
   </link>
@@ -276,9 +256,7 @@
     </collision> </xacro:unless>
     <inertial>
-      <mass value="0.242" />
-      <!--origin xyz="0 -0.02 0" rpy="0 -0 0"/>
-      <inertia ixx="0.000228" ixy="0" ixz="0" iyy="0.000148" iyz="0" izz="0.000263"/-->
-      <origin xyz="0 -0.02 0.015" rpy="0 -0 0"/>
-      <inertia ixx="0.00133" ixy="0" ixz="0" iyy="0.001" iyz="0" izz="0.00133"/>
+      <mass value="0.738" />
+      <origin xyz="0.0001 0.0499 0.0044" rpy="0 -0 0"/>
+      <inertia ixx="0.002" ixy="0" ixz="0" iyy="0.0003" iyz="0.0002" izz="0.0019"/>
     </inertial>
   </link>
@@ -298,8 +276,7 @@
     </collision> </xacro:unless>
     <inertial>
-      <mass value="0.744" />
-      <!--origin xyz="0 -0.01 0" rpy="0 -0 0"/-->
-      <origin xyz="0 0.01 -0.06" rpy="0 -0 0"/>
-      <inertia ixx="0.000841" ixy="0" ixz="0" iyy="0.000835" iyz="0" izz="0.000305"/>
+      <mass value="0.834" />
+      <origin xyz="-0.0007 0.0096 -0.0768" rpy="0 -0 0"/>
+      <inertia ixx="0.0011" ixy="0" ixz="0" iyy="0.0011" iyz="0" izz="0.0004"/>
     </inertial>
   </link>
@@ -319,10 +296,7 @@
     </collision> </xacro:unless>
     <inertial>
-      <mass value="0.574" />
-      <!--origin xyz="0.005 0 -0.0654" rpy="0 -0 0"/>
-      <inertia ixx="0.00114" ixy="0" ixz="0" iyy="0.00117" iyz="0" izz="0.000269"/-->
-      <!-- fix for gazebo -->
-      <origin xyz="0.005 0 -0.0654" rpy="0 -0 0"/>
-      <inertia ixx="0.00214" ixy="0" ixz="0" iyy="0.00217" iyz="0" izz="0.003"/>
+      <mass value="0.852" />
+      <origin xyz="-0.0099 0 -0.0496" rpy="0 -0 0"/>
+      <inertia ixx="0.0015" ixy="0" ixz="0.0001" iyy="0.0016" iyz="0" izz="0.0005"/>
     </inertial>
   </link>
@@ -342,10 +316,7 @@
     </collision> </xacro:unless>
     <inertial>
-      <mass value="0.711" />
-      <!--origin xyz="0.0047 0 -0.0546" rpy="0 -0 0"/>
-      <inertia ixx="0.00178" ixy="0" ixz="0" iyy="0.00179" iyz="0" izz="0.000273"/-->
-      <!-- fix for gazebo -->
-      <origin xyz="-0.03 0 -0.0546" rpy="0 -0 0"/>
-      <inertia ixx="0.00178" ixy="0" ixz="0" iyy="0.00179" iyz="0" izz="0.0035"/>
+      <mass value="0.251" />
+      <origin xyz="-0.0422 -0.0002 -0.0061" rpy="0 -0 0"/>
+      <inertia ixx="0.0005" ixy="0" ixz="0.0001" iyy="0.0005" iyz="0" izz="0.0002"/>
     </inertial>
   </link>
@@ -365,8 +336,7 @@
     </collision> </xacro:unless>
     <inertial>
-      <mass value="0.132" />
-      <origin xyz="0.006 0 -0.0738" rpy="0 -0 0"/>
-      <!--inertia ixx="0.00276" ixy="0" ixz="0" iyy="0.00286" iyz="0" izz="0.004"/-->
-      <inertia ixx="0.0007" ixy="0" ixz="0" iyy="0.0007" iyz="0" izz="0.0004"/>
+      <mass value="0.91" />
+      <origin xyz="0.0 -0.0018 -0.0754" rpy="0 -0 0"/>
+      <inertia ixx="0.0022" ixy="0" ixz="0" iyy="0.0023" iyz="0" izz="0.0004"/>
     </inertial>
   </link>
@@ -374,7 +344,7 @@
   <link name="r_wrist_center">
     <inertial>
-      <mass value="0.05" />
-      <origin xyz="0 0 0" rpy="0 -0 0"/>
-      <inertia ixx="0.0001" ixy="0" ixz="0" iyy="0.0001" iyz="0" izz="0.0001"/>
+      <mass value="0.005" />
+      <origin xyz="0 -0.0019 0" rpy="0 -0 0"/>
+      <inertia ixx="0.0" ixy="0" ixz="0" iyy="0.0" iyz="0" izz="0.0"/>
     </inertial>
   </link>
